Commit message: Changed the pioneed xacro file

File: src/pioneer_gazebo_ros/pioneer_description/urdf/pioneer3dx.xacro (robot description, xacro)
@@ -39,5 +39,5 @@
 <!-- Top -->
 	<joint name="base_top_joint" type="fixed">
-		<origin xyz="-0.045 0 0.234" rpy="0 0 0"/>
+		<origin xyz="0 0 0.234" rpy="0 0 0"/>
 		<parent link="base_link"/>
 		<child link="top_plate"/>
@@ -339,5 +339,5 @@
   </link>
   <joint name="camera_joint" type="fixed">
-    <origin xyz="0.17 0 0.0255" rpy="0 0 0"/>
+    <origin xyz="0 0 0.0255" rpy="0 0 0"/>
     <parent link="top_plate"/>
     <child link="camera_link"/>
